Commit message: feat: implement initial XACRO model for HUMANOIDTANAKA3 with evaluation and testing scripts

File: model/HUMANOIDTANAKA3.xacro (robot description, xacro)
@@ -1,7 +1,5 @@
 <?xml version="1.0" ?>
 <robot name="HUMANOIDTANAKA3" xmlns:xacro="http://www.ros.org/wiki/xacro">
-<xacro:include filename="$(find HUMANOIDTANAKA3_description)/urdf/materials.xacro" />
-<xacro:include filename="$(find HUMANOIDTANAKA3_description)/urdf/HUMANOIDTANAKA3.trans" />
-<xacro:include filename="$(find HUMANOIDTANAKA3_description)/urdf/HUMANOIDTANAKA3.gazebo" />
+<xacro:include filename="materials.xacro" />
 <link name="base_link">
   <inertial>
@@ -13,5 +11,5 @@
     <origin xyz="0 0 0" rpy="0 0 0"/>
     <geometry>
-      <mesh filename="package://HUMANOIDTANAKA3_description/meshes/base_link.stl" scale="0.001 0.001 0.001"/>
+      <mesh filename="meshes/base_link.stl" scale="0.001 0.001 0.001"/>
     </geometry>
     <material name="silver"/>
@@ -20,5 +18,5 @@
     <origin xyz="0 0 0" rpy="0 0 0"/>
     <geometry>
-      <mesh filename="package://HUMANOIDTANAKA3_description/meshes/base_link.stl" scale="0.001 0.001 0.001"/>
+      <mesh filename="meshes/base_link.stl" scale="0.001 0.001 0.001"/>
     </geometry>
   </collision>
@@ -33,5 +31,5 @@
     <origin xyz="0.009671 0.0387 0.128257" rpy="0 0 0"/>
     <geometry>
-      <mesh filename="package://HUMANOIDTANAKA3_description/meshes/Leg12_v1_1.stl" scale="0.001 0.001 0.001"/>
+      <mesh filename="meshes/Leg12_v1_1.stl" scale="0.001 0.001 0.001"/>
     </geometry>
     <material name="silver"/>
@@ -40,5 +38,5 @@
     <origin xyz="0.009671 0.0387 0.128257" rpy="0 0 0"/>
     <geometry>
-      <mesh filename="package://HUMANOIDTANAKA3_description/meshes/Leg12_v1_1.stl" scale="0.001 0.001 0.001"/>
+      <mesh filename="meshes/Leg12_v1_1.stl" scale="0.001 0.001 0.001"/>
     </geometry>
   </collision>
@@ -53,5 +51,5 @@
     <origin xyz="0.009671 -0.0387 0.128257" rpy="0 0 0"/>
     <geometry>
-      <mesh filename="package://HUMANOIDTANAKA3_description/meshes/Leg12_v1__1__1.stl" scale="0.001 0.001 0.001"/>
+      <mesh filename="meshes/Leg12_v1__1__1.stl" scale="0.001 0.001 0.001"/>
     </geometry>
     <material name="silver"/>
@@ -60,5 +58,5 @@
     <origin xyz="0.009671 -0.0387 0.128257" rpy="0 0 0"/>
     <geometry>
-      <mesh filename="package://HUMANOIDTANAKA3_description/meshes/Leg12_v1__1__1.stl" scale="0.001 0.001 0.001"/>
+      <mesh filename="meshes/Leg12_v1__1__1.stl" scale="0.001 0.001 0.001"/>
     </geometry>
   </collision>
@@ -73,5 +71,5 @@
     <origin xyz="0.009671 0.0387 -2.9e-05" rpy="0 0 0"/>
     <geometry>
-      <mesh filename="package://HUMANOIDTANAKA3_description/meshes/YAMAMOdogA.step_1.stl" scale="0.001 0.001 0.001"/>
+      <mesh filename="meshes/YAMAMOdogA.step_1.stl" scale="0.001 0.001 0.001"/>
     </geometry>
     <material name="silver"/>
@@ -80,5 +78,5 @@
     <origin xyz="0.009671 0.0387 -2.9e-05" rpy="0 0 0"/>
     <geometry>
-      <mesh filename="package://HUMANOIDTANAKA3_description/meshes/YAMAMOdogA.step_1.stl" scale="0.001 0.001 0.001"/>
+      <mesh filename="meshes/YAMAMOdogA.step_1.stl" scale="0.001 0.001 0.001"/>
     </geometry>
   </collision>
@@ -93,5 +91,5 @@
     <origin xyz="0.009671 0.0297 0.064114" rpy="0 0 0"/>
     <geometry>
-      <mesh filename="package://HUMANOIDTANAKA3_description/meshes/YAMAMOdogA.stepA_2.stl" scale="0.001 0.001 0.001"/>
+      <mesh filename="meshes/YAMAMOdogA.stepA_2.stl" scale="0.001 0.001 0.001"/>
     </geometry>
     <material name="silver"/>
@@ -100,5 +98,5 @@
     <origin xyz="0.009671 0.0297 0.064114" rpy="0 0 0"/>
     <geometry>
-      <mesh filename="package://HUMANOIDTANAKA3_description/meshes/YAMAMOdogA.stepA_2.stl" scale="0.001 0.001 0.001"/>
+      <mesh filename="meshes/YAMAMOdogA.stepA_2.stl" scale="0.001 0.001 0.001"/>
     </geometry>
   </collision>
@@ -113,5 +111,5 @@
     <origin xyz="0.009671 -0.0297 0.064114" rpy="0 0 0"/>
     <geometry>
-      <mesh filename="package://HUMANOIDTANAKA3_description/meshes/YAMAMOdogA.step_2.stl" scale="0.001 0.001 0.001"/>
+      <mesh filename="meshes/YAMAMOdogA.step_2.stl" scale="0.001 0.001 0.001"/>
     </geometry>
     <material name="silver"/>
@@ -120,5 +118,5 @@
     <origin xyz="0.009671 -0.0297 0.064114" rpy="0 0 0"/>
     <geometry>
-      <mesh filename="package://HUMANOIDTANAKA3_description/meshes/YAMAMOdogA.step_2.stl" scale="0.001 0.001 0.001"/>
+      <mesh filename="meshes/YAMAMOdogA.step_2.stl" scale="0.001 0.001 0.001"/>
     </geometry>
   </collision>
@@ -133,5 +131,5 @@
     <origin xyz="0.009671 -0.0387 -2.9e-05" rpy="0 0 0"/>
     <geometry>
-      <mesh filename="package://HUMANOIDTANAKA3_description/meshes/YAMAMOdogA.stepA_1.stl" scale="0.001 0.001 0.001"/>
+      <mesh filename="meshes/YAMAMOdogA.stepA_1.stl" scale="0.001 0.001 0.001"/>
     </geometry>
     <material name="silver"/>
@@ -140,5 +138,5 @@
     <origin xyz="0.009671 -0.0387 -2.9e-05" rpy="0 0 0"/>
     <geometry>
-      <mesh filename="package://HUMANOIDTANAKA3_description/meshes/YAMAMOdogA.stepA_1.stl" scale="0.001 0.001 0.001"/>
+      <mesh filename="meshes/YAMAMOdogA.stepA_1.stl" scale="0.001 0.001 0.001"/>
     </geometry>
   </collision>
