Commit message: chore: add humanoid model, test environment, and scripts for environment configuration and file cleanup

File: model/humanoid.urdf (robot description, URDF)
Before this commit: robot HUMANOIDTANAKA3, 7 links, 6 joints
Links:
- link Leg12_v1_1: mass 0.0 -> 0.5
- link Leg12_v1__1__1: mass 0.0 -> 0.5
- link base_link: mass 0.0 -> 0.5
