Commit message: 8サーボ(股ロール追加)の新設計に差し替え + 歩容学習の報酬・環境を改修
model/:
- humanoid.urdf/params.yaml/meshes を HumanoidTNK_FINAL (8DOF: 各脚 股ロール+股ピッチ+膝+足首ピッチ) に置換
- Fusionのマテリアル密度が鋼鉄設定で質量が約6.3倍だったため、STLから体積・重心・慣性を再計算
  (実効PLA密度1178 + MG996R x8 + 電装150g、総質量951g)。関節 effort/velocity を MG996R値(1.0N·m/6rad/s)に
- 旧6DOF資産(HUMANOIDTANAKA3.*, Leg12/YAMAMOdogAメッシュ, .bak)を削除、raw Fusion export を provenance用に追加
- 慣性テンソルは全リンク正定値+三角不等式を確認、PyBullet読込・自己干渉0を確認

learning/:
- 観測に base_linear_velocity 追加、足の接地/高さ/滑り/上下速度をセンシング
- WalkingReward: 速度追従・向き/横ズレ抑制・片足支持ボーナス・遊脚クリアランス・接地滑りペナルティ
- カリキュラムの num_joints バグ修正、報酬正規化オフ、entropy係数
- 足リンク名を新モデル(LU4_1/RU4_1)に、foot_rest_height を8DOF実測値0.014に

※ rewards.py の各重みは旧6DOF walk11(安定化途中)の値。8DOFでの再学習時に要調整。

Co-Authored-By: Claude Sonnet 5 <noreply@anthropic.com>

File: model/humanoid.urdf (robot description, URDF)
Before this commit: robot HUMANOIDTANAKA3, 7 links, 6 joints
Links:
- removed link Leg12_v1_1
- removed link Leg12_v1__1__1
- removed link YAMAMOdogA.stepA_1
- removed link YAMAMOdogA.stepA_2
- removed link YAMAMOdogA.step_1
- removed link YAMAMOdogA.step_2
- added link LU1_1, mass 0.09768; collision mesh filename=meshes/LU1_1.stl scale=0.001 0.001 0.001; visual mesh filename=meshes/LU1_1.stl scale=0.001 0.001 0.001
- added link LU2_1, mass 0.09861; collision mesh filename=meshes/LU2_1.stl scale=0.001 0.001 0.001; visual mesh filename=meshes/LU2_1.stl scale=0.001 0.001 0.001
- added link LU3_1, mass 0.09861; collision mesh filename=meshes/LU3_1.stl scale=0.001 0.001 0.001; visual mesh filename=meshes/LU3_1.stl scale=0.001 0.001 0.001
- added link LU4_1, mass 0.01280; collision mesh filename=meshes/LU4_1.stl scale=0.001 0.001 0.001; visual mesh filename=meshes/LU4_1.stl scale=0.001 0.001 0.001
- added link RU1_1, mass 0.09768; collision mesh filename=meshes/RU1_1.stl scale=0.001 0.001 0.001; visual mesh filename=meshes/RU1_1.stl scale=0.001 0.001 0.001
- added link RU2_1, mass 0.09861; collision mesh filename=meshes/RU2_1.stl scale=0.001 0.001 0.001; visual mesh filename=meshes/RU2_1.stl scale=0.001 0.001 0.001
- added link RU3_1, mass 0.09861; collision mesh filename=meshes/RU3_1.stl scale=0.001 0.001 0.001; visual mesh filename=meshes/RU3_1.stl scale=0.001 0.001 0.001
- added link RU4_1, mass 0.01280; collision mesh filename=meshes/RU4_1.stl scale=0.001 0.001 0.001; visual mesh filename=meshes/RU4_1.stl scale=0.001 0.001 0.001
- link base_link: mass 0.3522 -> 0.33595
Joints:
- removed joint joint_1
- removed joint joint_2
- removed joint joint_3
- removed joint joint_4
- removed joint joint_5
- removed joint joint_6
- added joint L_ankle_pitch: type revolute, parent LU3_1, child LU4_1, origin xyz=0.0175 0.0 -0.06445 rpy=0 0 0, axis 1.0 0.0 -0.0, limit lower=-1.570796 upper=1.570796 effort=1.0 velocity=6.0
- added joint L_hip_pitch: type revolute, parent LU1_1, child LU2_1, origin xyz=0.03975 -0.0507 -5e-05 rpy=0 0 0, axis 1.0 0.0 -0.0, limit lower=-1.570796 upper=1.570796 effort=1.0 velocity=6.0
- added joint L_hip_roll: type revolute, parent base_link, child LU1_1, origin xyz=-0.02 0.078 0.0001 rpy=0 0 0, axis 0.0 -1.0 -0.0, limit lower=-1.570796 upper=1.570796 effort=1.0 velocity=6.0
- added joint L_knee: type revolute, parent LU2_1, child LU3_1, origin xyz=-0.0175 0.0 -0.06445 rpy=0 0 0, axis 1.0 0.0 -0.0, limit lower=-1.570796 upper=1.570796 effort=1.0 velocity=6.0
- added joint R_ankle_pitch: type revolute, parent RU3_1, child RU4_1, origin xyz=-0.0175 0.0 -0.06445 rpy=0 0 0, axis -1.0 0.0 0.0, limit lower=-1.570796 upper=1.570796 effort=1.0 velocity=6.0
- added joint R_hip_pitch: type revolute, parent RU1_1, child RU2_1, origin xyz=-0.03975 -0.0507 -5e-05 rpy=0 0 0, axis -1.0 0.0 0.0, limit lower=-1.570796 upper=1.570796 effort=1.0 velocity=6.0
- added joint R_hip_roll: type revolute, parent base_link, child RU1_1, origin xyz=-0.05 0.078 0.0001 rpy=0 0 0, axis 0.0 -1.0 -0.0, limit lower=-1.570796 upper=1.570796 effort=1.0 velocity=6.0
- added joint R_knee: type revolute, parent RU2_1, child RU3_1, origin xyz=0.0175 0.0 -0.06445 rpy=0 0 0, axis 1.0 0.0 0.0, limit lower=-1.570796 upper=1.570796 effort=1.0 velocity=6.0

File: model/materials.xacro (robot description, xacro)
@@ -1,4 +1,4 @@
 <?xml version="1.0" ?>
-<robot name="HUMANOIDTANAKA3" xmlns:xacro="http://www.ros.org/wiki/xacro" >
+<robot name="HumanoidTNK_FINAL" xmlns:xacro="http://www.ros.org/wiki/xacro" >
 <material name="silver">
   <color rgba="0.700 0.700 0.700 1.000"/>

Commit message: 参照歩容 + 残差RLで8DOF歩行を獲得
PyBullet 上で、左右の足を交互に上げて歩く歩容を獲得した。
20s×10 で転倒 0/10、0.128 m/s、3N の外乱を受けても転倒 0/10。

- model/reference_gait.yaml: 探索で見つけた開ループ参照歩容（周期 0.523s）
- model/params_residual.yaml + learning/train/curriculum_residual.yaml:
  関節目標角 = 参照歩容 + 残差(±0.15〜0.25rad) の残差 PPO 設定
- base_env / pybullet_env: 歩行位相クロックを観測に追加（2N+12次元）、
  参照歩容+残差制御、足以外の接地検出、足の前後速度
- rewards: 位相追従・座り込み/胴体接地での終了・速度ゲート・
  離地バランスなど、学習中に見つかった抜け道への対策
- train.py: --start-phase / --log-std-init、開始フェーズ報酬の適用漏れを修正
- learning/eval: gait_metrics（歩容の数値評価）、gait_search（参照歩容探索）、
  record_video（MP4 書き出し）
- 学習済みモデルは Git に入れず learning/policies/README.md に索引を記載

Co-Authored-By: Claude Opus 5.5 <noreply@anthropic.com>

File: model/humanoid.urdf (robot description, URDF)
Before this commit: robot HumanoidTNK_FINAL, 9 links, 8 joints
Joints:
- joint R_knee: axis 1.0 0.0 0.0 -> -1.0 0.0 0.0
